Commit message: 2022/12/18

File: Models/bowl_target.urdf (robot description, URDF)
Before this commit: robot bowl, 1 links, 0 joints
Links:
- link baseLink: geometry collision mesh filename=D:\code\Dynamic-Grasping\Models\bowl\bowl.obj; visual mesh filename=D:\code\Dynamic-Grasping\Models\bowl\bowl.obj

File: Models/cube_target.urdf (robot description, URDF)
Before this commit: robot cube, 1 links, 0 joints
Links:
- link baseLink: geometry collision mesh filename=D:\code\Dynamic-Grasping\Models\cube\cube.obj; visual mesh filename=D:\code\Dynamic-Grasping\Models\cube\cube.obj
