Commit message: 3-13-1

File: Models/mug_target.urdf (robot description, URDF)
Before this commit: robot mug, 1 links, 0 joints
Links:
- link baseLink: mass 5.01 -> 1.01; geometry collision mesh filename=D:\code\Dynamic-Grasping\Models\mug\mug.obj; visual mesh filename=D:\code\Dynamic-Grasping\Models\mug\mug.obj
